File: picoflutter/picoflutter.kicad_sch (KiCad schematic)
At the start: 67 parts, among them IC1 AP7361EA-33E-13, IC3 W25Q64JVZPIQ, J2 SM04B-SRSS-TB, J4 S2B-PH-SM4-TB(LF)(SN), J5 USB4105-GF-A, Q1 DMG3415, SW2 MK-12C02-G020, U1 MCP73831T-2ACI/OT, U3 RP2040, Y1 445I23D12M00000

Commit message: Move README to repo root, remove generated ibom, KiCad resave
Claude-Session: https://claude.ai/code/session_01CTpVuugoA5qMQu3t31zp5N
Parts:
- C1, C2: value 4.7u -> (none)
- C10, C12, C13, C14, C15, C16, C17, C3, C7, C8: value 100n -> (none)
- C11, C9: value 1u -> (none)
- C20, C6: value 10uF -> (none)
- C4, C5: value 27p -> (none)
- CHG1: value ORANGE -> (none)
- D2: value MBR0540 -> (none)
- IC1: value AP7361EA-33E-13 -> (none)
- IC3: value W25Q64JVZPIQ -> (none)
- J2: value SM04B-SRSS-TB -> (none)
- J4: value S2B-PH-SM4-TB(LF)(SN) -> (none)
- J5: value USB4105-GF-A -> (none)
- LED1, LED10, LED11, LED12, LED13, LED14, LED15, LED16, LED17, LED18, LED19, LED2, LED20, LED21, LED22, LED23, LED24, LED25, LED26, LED3, LED4, LED5, LED6, LED7, LED8, LED9: value 1010RGBC-WS2812B -> (none)
- Q1: value DMG3415 -> (none)
- R1, R5: value 10K -> (none)
- R2: value 5.1K -> (none)
- R26, R27: value 1k -> (none)
- R28: value DNF -> (none)
- R29, R30: value 27 -> (none)
- R3, R4: value 5k1 -> (none)
- S1: value TS-1088-AR02016 -> (none)
- SW2: value MK-12C02-G020 -> (none)
- U1: value MCP73831T-2ACI/OT -> (none)
- U3: value RP2040 -> (none)
- Y1: value 445I23D12M00000 -> (none)
